Commit message: Add files via upload

File: urdf/slam_project.urdf.xacro (robot description, xacro)
@@ -0,0 +1,51 @@
+<?xml version="1.0"?>
+<robot name="slam_project" xmlns:xacro="http://ros.org/wiki/xacro">
+  <xacro:macro name="turtlebot_sim_3dsensor">
+  <!-- RGBD Camera -->
+  <gazebo reference="camera_link">
+    <sensor type="depth" name="camera1">
+        <always_on>1</always_on>
+        <update_rate>20.0</update_rate>
+        <visualize>true</visualize>
+        <camera>
+           <pose>0 0 0 pi 0 0</pose>
+           <horizontal_fov>1.047</horizontal_fov>
+            <image>
+                <width>640</width>
+                <height>480</height>
+                <format>R8G8B8</format>
+            </image>
+            <depth_camera>
+				<!-- not used... -->
+            </depth_camera>
+            <clip>
+                <near>0.1</near>
+                <far>20</far>
+            </clip>
+        </camera>
+        <plugin name="camera_controller" filename="libgazebo_ros_openni_kinect.so">
+		<alwaysOn>true</alwaysOn>
+		<updateRate>10.0</updateRate>
+		<cameraName>camera</cameraName>
+		<frameName>camera_rgbd_frame</frameName>
+		<imageTopicName>rgb/image_raw</imageTopicName>
+		<depthImageTopicName>depth/image_raw</depthImageTopicName>
+		<pointCloudTopicName>depth/points</pointCloudTopicName>
+		<cameraInfoTopicName>rgb/camera_info</cameraInfoTopicName>
+		<depthImageCameraInfoTopicName>depth/camera_info</depthImageCameraInfoTopicName>
+		<pointCloudCutoff>0.4</pointCloudCutoff>
+		<hackBaseline>0.07</hackBaseline>
+		<distortionK1>0.0</distortionK1>
+		<distortionK2>0.0</distortionK2>
+		<distortionK3>0.0</distortionK3>
+		<distortionT1>0.0</distortionT1>
+		<distortionT2>0.0</distortionT2>
+		<CxPrime>0.0</CxPrime>
+		<Cx>0.0</Cx>
+		<Cy>0.0</Cy>
+		<focalLength>0.0</focalLength>
+	</plugin>
+    </sensor>
+  </gazebo>
+  </xacro:macro>
+</robot>
